File: hardware/E-IEC-Nano-SRAM/4-layer/64korppu-E.kicad_pcb (KiCad board)
At the start: 4 copper layers, 70 x 60 mm, 27 parts, among them J1 DIN-6_IEC, J2 Floppy_34pin, J3 DC_Jack, U1 Arduino_Nano, U2 23LC1024, U3 74HC595

Commit message: Fix 4-layer PCB: all nets connected, 0 critical DRC errors
- Add manual +5V traces: U2.7→U2.8 (F.Cu), R12.1→R11.1 (F.Cu),
  U3.16→R12.1 (B.Cu routed around FLOPPY_DIR via)
- DRC result: 0 critical, 0 unconnected, 0 shorts
- Only cosmetic warnings remain (silk_over_copper)

Co-Authored-By: Claude Opus 4.6 <noreply@anthropic.com>
Routing:
- net +5V: track 0.00 -> 22.2 mm
