File: hardware/E-IEC-Nano-SRAM/4-layer/64korppu-E.kicad_pcb (KiCad board)
At the start: 4 copper layers, 70 x 60 mm, 41 parts, among them J1 DIN-6_IEC, J2 Floppy_34pin, J3 DC_Jack, U1 Arduino_Nano, U2 23LC256, U3 74HC595

Commit message: Add "C64 HD Floppy Controller" title to board label
Label now reads: C64 HD Floppy Controller / karski by / design 2026 / rev 001.
Updated on both 2-layer and 4-layer PCBs, resize script, and gerbers.

Co-Authored-By: Claude Opus 4.6 <noreply@anthropic.com>
Other:
- board text added: "C64 HD Floppy Controller karski by design 2026 rev 001"
- board text removed: "karski by design 2026 rev 001"
Changed lines of the file:
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@@
 		(layer "Edge.Cuts")
 	)
-	(gr_text "karski by\ndesign 2026\nrev 001"
+	(gr_text "C64 HD Floppy Controller\nkarski by\ndesign 2026\nrev 001"
 		(at 118 113.5 0)
 		(layer "F.SilkS")
